Commit message: Parte12

File: Parte12/robutler_description/urdf/common_properties.xacro (robot description, xacro)
@@ -13,4 +13,7 @@
   <material name="blue">
     <color rgba="0.0 0.0 0.8 1.0"/>
+  </material>
+  <material name="turquoise">
+    <color rgba="0 0.808 0.82 1.0"/>
   </material>
   <material name="green">

File: Parte12/robutler_description/urdf/robutler.gazebo.xacro (robot description, xacro)
@@ -5,5 +5,6 @@
   <xacro:arg name="imu_visual"    default="false"/>
   <gazebo reference="base_link">
-    <material>Gazebo/DarkGrey</material>
+    <!-- <material>Gazebo/DarkGrey</material> -->
+    <material>Gazebo/Turquoise</material>
   </gazebo>
   <gazebo reference="wheel_left_link">

File: Parte12/robutler_description/urdf/robutler.urdf.xacro (robot description, xacro)
@@ -15,5 +15,6 @@
         <mesh filename="package://turtlebot3_description/meshes/bases/waffle_pi_base.stl" scale="0.001 0.001 0.001"/>
       </geometry>
-      <material name="light_black"/>
+      <!-- <material name="light_black"/> -->
+      <material name="turquoise"/>
     </visual>
     <collision>
@@ -162,5 +163,5 @@
   <joint name="camera_joint" type="fixed">
     <!-- <origin xyz="0.073 -0.011 0.084" rpy="0 0 0"/> -->
-    <origin xyz="0.073 -0.011 0.484" rpy="0 0 0"/>
+    <origin xyz="0.073 -0.011 1" rpy="0 0 0"/>
     <parent link="base_link"/>
     <child link="camera_link"/>
